Commit message: add urdf gen yaml

File: maniptrans_envs/assets/inspire_hand/inspire_hand_right.urdf (robot description, URDF)
Before this commit: robot h1, 18 links, 17 joints
Links:
- link R_hand_base_link: geometry collision box size=0.01 0.1 0.05; visual box size=0.01 0.1 0.05
- link R_index_intermediate: geometry collision box size=0.01 0.04379631116135011 0.01; visual box size=0.01 0.04379631116135011 0.01
- link R_index_proximal: geometry collision box size=0.01 0.03214804234226402 0.01; visual box size=0.01 0.03214804234226402 0.01
- link R_index_tip: geometry visual sphere radius=0.006999999999999999
- link R_middle_intermediate: geometry collision box size=0.01 0.04706433173139187 0.01; visual box size=0.01 0.04706433173139187 0.01
- link R_middle_proximal: geometry collision box size=0.01 0.03214803454972014 0.01; visual box size=0.01 0.03214803454972014 0.01
- link R_middle_tip: geometry visual sphere radius=0.006999999999999999
- link R_pinky_intermediate: geometry collision box size=0.01 0.03671467408620836 0.01; visual box size=0.01 0.03671467408620836 0.01
- link R_pinky_proximal: geometry collision box size=0.01 0.03214803454972014 0.01; visual box size=0.01 0.03214803454972014 0.01
- link R_pinky_tip: geometry visual sphere radius=0.006999999999999999
- link R_ring_intermediate: geometry collision box size=0.01 0.04379633523392682 0.01; visual box size=0.01 0.04379633523392682 0.01
- link R_ring_proximal: geometry collision box size=0.01 0.03214803454972014 0.01; visual box size=0.01 0.03214803454972014 0.01
- link R_ring_tip: geometry visual sphere radius=0.006999999999999999
- link R_thumb_distal: geometry collision box size=0.01 0.023078574950895474 0.01; visual box size=0.01 0.023078574950895474 0.01
- link R_thumb_intermediate: geometry collision box size=0.01 0.02268404373122217 0.01; visual box size=0.01 0.02268404373122217 0.01
- link R_thumb_proximal: geometry collision box size=0.01 0.056006380966814845 0.01; visual box size=0.01 0.056006380966814845 0.01
- link R_thumb_proximal_base: geometry collision box size=0.01 0.016787272024066328 0.01; visual box size=0.01 0.016787272024066328 0.01
- link R_thumb_tip: geometry visual sphere radius=0.006999999999999999
Joints:
- joint R_index_intermediate_joint: origin xyz=-0.0026138 0.032026 -0.001 rpy=0 0 0 -> xyz=0 0.032026 0 rpy=0 0 0
- joint R_index_tip_joint: origin xyz=-0.00412053 0.0433132 -0.00501047 rpy=0 0 0 -> xyz=-0.005 0.0433132 -0.005 rpy=0 0 0
- joint R_middle_intermediate_joint: origin xyz=-0.0024229 0.032041 -0.001 rpy=0 0 0 -> xyz=0 0.032041 0 rpy=0 0 0
- joint R_middle_tip_joint: origin xyz=-0.00426879 0.0466043 -0.00498678 rpy=0 0 0 -> xyz=-0.005 0.0466043 -0.005 rpy=0 0 0
- joint R_pinky_intermediate_joint: origin xyz=-0.0024229 0.032041 -0.001 rpy=0 0 0 -> xyz=0 0.032041 0 rpy=0 0 0
- joint R_pinky_tip_joint: origin xyz=-0.00260734 0.0362776 -0.00501047 rpy=0 0 0 -> xyz=-0.005 0.0362776 -0.005 rpy=0 0 0
- joint R_ring_intermediate_joint: origin xyz=-0.0024229 0.032041 -0.001 rpy=0 0 0 -> xyz=0 0.032041 0 rpy=0 0 0
- joint R_ring_tip_joint: origin xyz=-0.00366554 0.0433541 -0.00501047 rpy=0 0 0 -> xyz=-0.005 0.0433541 -0.005 rpy=0 0 0
- joint R_thumb_tip_joint: origin xyz=0.0159104 0.0156076 -0.00599021 rpy=0 0 0 -> xyz=0.020 0.012 -0.0020 rpy=0 0 0
